Commit message: Add contact force reward term. Pass in urdf from config.

File: panda_isaac/asset/urdf/franka_description/robots/franka_panda_cam.urdf (robot description, URDF)
Before this commit: robot panda, 11 links, 10 joints
Links:
- added link camera; collision box size=0.026 0.124 0.029; visual box size=0.026 0.124 0.029
Joints:
- added joint camera_joint_fixed: type fixed, parent panda_hand, child camera, origin xyz=0 0 0 rpy=0 0 0
